File: digital_clock/layouts/default/default.kicad_pcb (KiCad board)
At the start: 2 copper layers, 1 part

Commit message: add lesson in README
Parts:
- removed SW1: , ShiftReg:SOIC-16_3.9x9.9mm_P1.27mm
